Commit message: Fix PID error

File: urdf/xmobot_base.xacro (robot description, xacro)
@@ -11,5 +11,5 @@
         <parent link="base_footprint"/>
         <child link="base_link"/>
-        <origin xyz="0 0 ${robot_height/2}" rpy="0 0 0"/>
+        <origin xyz="0 0 ${wheel_radius*2}" rpy="0 0 0"/>
     </joint>
     <link name="base_link">
@@ -35,5 +35,5 @@
             </geometry>
         </collision>
-        <xacro:inertial_box mass="500" size_x="${robot_length}" size_y="${robot_width}" size_z="${robot_height}"/>
+        <xacro:inertial_box mass="5" size_x="${robot_length}" size_y="${robot_width}" size_z="${robot_height}"/>
     </link>
     <!-- 底盘结构 -->

File: urdf/xmobot_drive.xacro (robot description, xacro)
@@ -29,5 +29,5 @@
                         </geometry>
                     </collision>
-                    <xacro:inertial_cylinder mass="10" radius="0.05" length="0.03"/>
+                    <xacro:inertial_cylinder mass="0.5" radius="0.05" length="0.03"/>
                 </link>
                 <joint name="${prefix}_steering_joint" type="revolute">
@@ -63,11 +63,5 @@
                     </geometry>
                 </collision>
-                <inertial>
-                    <origin xyz="0 0 0" rpy="${M_PI_2} 0 0"/>  <!-- 注意这里也旋转M_PI_2 -->
-                    <mass value="5.0"/>
-                    <inertia
-                            ixx="1.0" iyy="1.0" izz="1.0"
-                            ixy="0.0" ixz="0.0" iyz="0.0"/>
-                </inertial>
+                <xacro:inertial_cylinder mass="5" radius="${wheel_radius}" length="${wheel_width}"/>
             </link>
             <!-- wheel joint -->

File: urdf/xmobot_gazebo.xacro (robot description, xacro)
@@ -194,9 +194,8 @@
         <gazebo reference="${wheel_link_name}">
             <material>Gazebo/DarkGrey</material>
-            <kp>100000.0</kp>
+            <kp>1e6</kp>
             <kd>1.0</kd>
             <mu1>1.0</mu1>
             <mu2>1.0</mu2>
-            <maxVel>1.0</maxVel>
             <minDepth>0.01</minDepth>
         </gazebo>
