Commit message: add a simple world

File: urdf/xmobot_drive.xacro (robot description, xacro)
@@ -63,5 +63,5 @@
                     </geometry>
                 </collision>
-                <xacro:inertial_cylinder mass="5" radius="${wheel_radius}" length="${wheel_width}"/>
+                <xacro:inertial_cylinder mass="1" radius="${wheel_radius}" length="${wheel_width}"/>
             </link>
             <!-- wheel joint -->
@@ -72,4 +72,5 @@
                     <origin xyz="0 0 ${-wheel_radius}" rpy="0 0 0"/>
                     <axis xyz="0 1 0"/>
+                    <limit effort="30.0" velocity="10.0"/>
                 </joint>
             </xacro:if>
@@ -80,4 +81,5 @@
                     <origin xyz="${x} ${y} ${-wheel_radius}" rpy="0 0 0"/>
                     <axis xyz="0 1 0"/>
+                    <limit effort="30.0" velocity="10.0"/>
                 </joint>
             </xacro:unless>

File: urdf/xmobot_gazebo.xacro (robot description, xacro)
@@ -153,13 +153,14 @@
             <implicitSpringDamper>1</implicitSpringDamper>
         </gazebo>
-<!--        <gazebo>-->
-<!--            <plugin name="object_controller" filename="libgazebo_ros_planar_move.so">-->
-<!--                <commandTopic>cmd_vel</commandTopic>-->
-<!--                <odometryTopic>odom</odometryTopic>-->
-<!--                <odometryFrame>odom</odometryFrame>-->
-<!--                <odometryRate>20.0</odometryRate>-->
-<!--                <robotBaseFrame>base_footprint</robotBaseFrame>-->
-<!--            </plugin>-->
-<!--        </gazebo>-->
+        <gazebo>
+            <plugin name="object_controller" filename="libgazebo_ros_planar_move.so">
+                <commandTopic>cmd_vel</commandTopic>
+                <odometryTopic>odom</odometryTopic>
+                <odometryFrame>odom</odometryFrame>
+                <odometryRate>20.0</odometryRate>
+                <cmdTimeout>0.25</cmdTimeout>
+                <robotBaseFrame>base_footprint</robotBaseFrame>
+            </plugin>
+        </gazebo>
         <!-- 测试用 -->
     </xacro:macro>
@@ -196,6 +197,6 @@
             <kp>1e6</kp>
             <kd>1.0</kd>
-            <mu1>1.0</mu1>
-            <mu2>1.0</mu2>
+            <mu1>1.2</mu1>
+            <mu2>0.8</mu2>
             <minDepth>0.01</minDepth>
         </gazebo>
