Commit message: Update README: Add known issues, debug commands, and refine Quick Start guide

File: urdf/xmobot.urdf.xacro (robot description, xacro)
@@ -1,4 +1,28 @@
 <?xml version="1.0"?>
-<robot xmlns:xacro="http://ros.org/wiki/xacro">
+<robot xmlns:xacro="http://www.ros.org/wiki/xacro" name="xmobot">
+    <!-- Define parameters with default values -->
+    <xacro:arg name="robot_length" default="0.5"/>
+    <xacro:arg name="robot_width" default="0.4"/>
+    <xacro:arg name="robot_height" default="0.1"/>
+    <xacro:arg name="wheel_radius" default="0.08"/>
+    <xacro:arg name="wheel_width" default="0.05"/>
+    <xacro:arg name="wheel_separation_x" default="0.5"/>
+    <xacro:arg name="wheel_separation_y" default="0.4"/>
+    <xacro:arg name="drive_type" default="4wis"/>
+    <xacro:arg name="use_mesh" default="false"/>
+    <!-- 全局参数 -->
+    <xacro:property name="use_mesh" value="$(arg use_mesh)"/>
+    <xacro:property name="drive_type" value="$(arg drive_type)"/>
+    <xacro:property name="robot_length" value="$(arg robot_length)" />
+    <xacro:property name="robot_width" value="$(arg robot_width)" />
+    <xacro:property name="robot_height" value="$(arg robot_height)" />
+    <xacro:property name="wheel_radius" value="$(arg wheel_radius)"/>
+    <xacro:property name="wheel_width" value="$(arg wheel_width)" />
+    <xacro:property name="wheel_separation_x" value="$(arg wheel_separation_x)" />
+    <xacro:property name="wheel_separation_y" value="$(arg wheel_separation_y)" />
+    <xacro:property name="M_PI" value="3.1415926535897931" />
+    <xacro:property name="M_PI_2" value="1.570796327" />
+    <xacro:property name="DEG_TO_RAD" value="0.017453293" />
+    <!-- Import Xacro -->
     <xacro:include filename="$(find xmobot)/urdf/xmobot_base.xacro"/>
 </robot>

File: urdf/xmobot_drive.xacro (robot description, xacro)
@@ -1,46 +1,120 @@
 <?xml version="1.0"?>
 <robot xmlns:xacro="http://ros.org/wiki/xacro">
-    <xacro:property name="drive_type" value="diff_drive"/>
-    <!-- diff_drive / ackermann / 4wis -->
-    <!-- Wheel distance parameters -->
-    <xacro:property name="wheel_separation_x" value="0.5"/>
-    <xacro:property name="wheel_separation_y" value="0.4"/>
-    <!-- Import wheel macro -->
-    <xacro:include filename="$(find xmobot)/urdf/xmobot_wheel.xacro"/>
     <xacro:macro name="drive_system">
+        <!-- 定义四个轮子的生成方式 -->
+        <xacro:macro name="wheel_unit" params="prefix x y enable_steer">
+            <!-- 如果需要加转向 -->
+            <xacro:if value="${enable_steer}">
+                <link name="${prefix}_steering_link">
+                    <visual>
+                        <origin xyz="0 0 0" rpy="0 0 0"/>
+                        <xacro:if value="${use_mesh}">
+                            <geometry>
+                                <mesh filename="package://xmobot/meshes/steering_link.dae" scale="1 1 1"/>
+                            </geometry>
+                        </xacro:if>
+                        <xacro:unless value="${use_mesh}">
+                            <geometry>
+                                <cylinder radius="0.05" length="0.03"/>
+                            </geometry>
+                        </xacro:unless>
+                        <material name="Gray">
+                            <color rgba="0.5 0.5 0.5 1.0"/>
+                        </material>
+                    </visual>
+                    <collision>
+                        <origin xyz="0 0 0" rpy="0 0 0"/>
+                        <geometry>
+                            <cylinder radius="0.05" length="0.03"/>
+                        </geometry>
+                    </collision>
+                    <xacro:inertial_cylinder mass="10" radius="0.05" length="0.03"/>
+                </link>
+                <joint name="${prefix}_steering_joint" type="revolute">
+                    <parent link="base_link"/>
+                    <child link="${prefix}_steering_link"/>
+                    <origin xyz="${x} ${y} 0" rpy="0 0 0"/>
+                    <axis xyz="0 0 1"/>
+                    <limit lower="${-90*DEG_TO_RAD}" upper="${90*DEG_TO_RAD}" effort="1.0" velocity="1.0"/>
+                </joint>
+            </xacro:if>
+            <!-- 轮子link -->
+            <link name="${prefix}_wheel_link">
+                <visual>
+                    <origin xyz="0 0 0" rpy="${M_PI_2} 0 0"/>
+                    <xacro:if value="${use_mesh}">
+                        <geometry>
+                            <mesh filename="package://xmobot/meshes/wheel.dae" scale="1 1 1"/>
+                        </geometry>
+                    </xacro:if>
+                    <xacro:unless value="${use_mesh}">
+                        <geometry>
+                            <cylinder radius="${wheel_radius}" length="${wheel_width}"/>
+                        </geometry>
+                    </xacro:unless>
+                    <material name="Black">
+                        <color rgba="0.1 0.1 0.1 1.0"/>
+                    </material>
+                </visual>
+                <collision>
+                    <origin xyz="0 0 0" rpy="${M_PI_2} 0 0"/>
+                    <geometry>
+                        <cylinder radius="${wheel_radius}" length="${wheel_width}"/>
+                    </geometry>
+                </collision>
+                <inertial>
+                    <origin xyz="0 0 0" rpy="${M_PI_2} 0 0"/>  <!-- 注意这里也旋转M_PI_2 -->
+                    <mass value="5.0"/>
+                    <inertia
+                            ixx="1.0" iyy="1.0" izz="1.0"
+                            ixy="0.0" ixz="0.0" iyz="0.0"/>
+                </inertial>
+            </link>
+            <!-- wheel joint -->
+            <xacro:if value="${enable_steer}">
+                <joint name="${prefix}_wheel_joint" type="continuous">
+                    <parent link="${prefix}_steering_link"/>
+                    <child link="${prefix}_wheel_link"/>
+                    <origin xyz="0 0 ${-wheel_radius}" rpy="0 0 0"/>
+                    <axis xyz="0 1 0"/>
+                </joint>
+            </xacro:if>
+            <xacro:unless value="${enable_steer}">
+                <joint name="${prefix}_wheel_joint" type="continuous">
+                    <parent link="base_link"/>
+                    <child link="${prefix}_wheel_link"/>
+                    <origin xyz="${x} ${y} ${-wheel_radius}" rpy="0 0 0"/>
+                    <axis xyz="0 1 0"/>
+                </joint>
+            </xacro:unless>
+        </xacro:macro>
+        <!-- 根据drive_type生成四个轮子 -->
         <xacro:if value="${drive_type == 'diff_drive' or drive_type == 'mecanum'}">
-            <!-- Four wheels directly attached to base_link -->
-            <xacro:wheel prefix="front_left"  mesh_file="package://xmobot/meshes/wheel.dae"/>
-            <joint name="front_left_wheel_joint" type="continuous">
-                <parent link="base_link"/>
-                <child link="front_left_wheel_link"/>
-                <origin xyz="${wheel_separation_x/2} ${wheel_separation_y/2} 0" rpy="0 0 0"/>
-                <axis xyz="0 1 0"/>
-            </joint>
-            <xacro:wheel prefix="front_right" mesh_file="package://xmobot/meshes/wheel.dae"/>
-            <joint name="front_right_wheel_joint" type="continuous">
-                <parent link="base_link"/>
-                <child link="front_right_wheel_link"/>
-                <origin xyz="${wheel_separation_x/2} ${-wheel_separation_y/2} 0" rpy="0 0 0"/>
-                <axis xyz="0 1 0"/>
-            </joint>
-            <xacro:wheel prefix="rear_left" mesh_file="package://xmobot/meshes/wheel.dae"/>
-            <joint name="rear_left_wheel_joint" type="continuous">
-                <parent link="base_link"/>
-                <child link="rear_left_wheel_link"/>
-                <origin xyz="${-wheel_separation_x/2} ${wheel_separation_y/2} 0" rpy="0 0 0"/>
-                <axis xyz="0 1 0"/>
-            </joint>
-            <xacro:wheel prefix="rear_right" mesh_file="package://xmobot/meshes/wheel.dae"/>
-            <joint name="rear_right_wheel_joint" type="continuous">
-                <parent link="base_link"/>
-                <child link="rear_right_wheel_link"/>
-                <origin xyz="${-wheel_separation_x/2} ${-wheel_separation_y/2} 0" rpy="0 0 0"/>
-                <axis xyz="0 1 0"/>
-            </joint>
+            <!-- 差速 / 麦克纳姆模式，四轮固定，不转向 -->
+            <xacro:wheel_unit prefix="front_left"  x="${wheel_separation_x/2}"  y="${wheel_separation_y/2}"  enable_steer="false"/>
+            <xacro:wheel_unit prefix="front_right" x="${wheel_separation_x/2}"  y="${-wheel_separation_y/2}" enable_steer="false"/>
+            <xacro:wheel_unit prefix="rear_left"   x="${-wheel_separation_x/2}" y="${wheel_separation_y/2}"  enable_steer="false"/>
+            <xacro:wheel_unit prefix="rear_right"  x="${-wheel_separation_x/2}" y="${-wheel_separation_y/2}" enable_steer="false"/>
         </xacro:if>
-        <xacro:if value="${drive_type == 'ackermann' or drive_type == '4wis'}">
-            <!-- 这里后续增加转向关节，双层嵌套 -->
-            <!-- （我们下一步细化四轮转向版本！） -->
+        <xacro:if value="${drive_type == 'ackermann_front'}">
+            <!-- 前轮转向阿克曼模式 -->
+            <xacro:wheel_unit prefix="front_left"  x="${wheel_separation_x/2}"  y="${wheel_separation_y/2}"  enable_steer="true"/>
+            <xacro:wheel_unit prefix="front_right" x="${wheel_separation_x/2}"  y="${-wheel_separation_y/2}" enable_steer="true"/>
+            <xacro:wheel_unit prefix="rear_left"   x="${-wheel_separation_x/2}" y="${wheel_separation_y/2}"  enable_steer="false"/>
+            <xacro:wheel_unit prefix="rear_right"  x="${-wheel_separation_x/2}" y="${-wheel_separation_y/2}" enable_steer="false"/>
+        </xacro:if>
+        <xacro:if value="${drive_type == 'ackermann_rear'}">
+            <!-- 后轮转向阿克曼模式 -->
+            <xacro:wheel_unit prefix="front_left"  x="${wheel_separation_x/2}"  y="${wheel_separation_y/2}"  enable_steer="false"/>
+            <xacro:wheel_unit prefix="front_right" x="${wheel_separation_x/2}"  y="${-wheel_separation_y/2}" enable_steer="false"/>
+            <xacro:wheel_unit prefix="rear_left"   x="${-wheel_separation_x/2}" y="${wheel_separation_y/2}"  enable_steer="true"/>
+            <xacro:wheel_unit prefix="rear_right"  x="${-wheel_separation_x/2}" y="${-wheel_separation_y/2}" enable_steer="true"/>
+        </xacro:if>
+        <xacro:if value="${drive_type == '4wis'}">
+            <!-- 四轮独立转向 -->
+            <xacro:wheel_unit prefix="front_left"  x="${wheel_separation_x/2}"  y="${wheel_separation_y/2}"  enable_steer="true"/>
+            <xacro:wheel_unit prefix="front_right" x="${wheel_separation_x/2}"  y="${-wheel_separation_y/2}" enable_steer="true"/>
+            <xacro:wheel_unit prefix="rear_left"   x="${-wheel_separation_x/2}" y="${wheel_separation_y/2}"  enable_steer="true"/>
+            <xacro:wheel_unit prefix="rear_right"  x="${-wheel_separation_x/2}" y="${-wheel_separation_y/2}" enable_steer="true"/>
         </xacro:if>
     </xacro:macro>

File: urdf/xmobot_sensors.xacro (robot description, xacro)
@@ -1,5 +1,5 @@
 <?xml version="1.0"?>
 <robot xmlns:xacro="http://ros.org/wiki/xacro">
-    <xacro:property name="lidar_height" value="0.05"/>
+    <xacro:property name="lidar_height" value="0.08"/>
     <xacro:property name="camera_height" value="0.0"/>
     <xacro:property name="camera_offset_x" value="0.3"/>
@@ -8,7 +8,15 @@
         <link name="lidar_link">
             <visual>
-                <geometry>
-                    <cylinder length="0.05" radius="0.05"/>
-                </geometry>
+                <origin xyz="0 0 0" rpy="0 0 0"/>
+                <xacro:if value="${use_mesh}">
+                    <geometry>
+                        <mesh filename="package://xmobot/meshes/lidar.dae" scale="1 1 1"/>
+                    </geometry>
+                </xacro:if>
+                <xacro:unless value="${use_mesh}">
+                    <geometry>
+                        <cylinder length="0.05" radius="0.05"/>
+                    </geometry>
+                </xacro:unless>
                 <material name="Blue">
                     <color rgba="0 0 1 1"/>
@@ -24,7 +32,15 @@
         <link name="camera_link">
             <visual>
-                <geometry>
-                    <box size="0.05 0.05 0.05"/>
-                </geometry>
+                <origin xyz="0 0 0" rpy="0 0 0"/>
+                <xacro:if value="${use_mesh}">
+                    <geometry>
+                        <mesh filename="package://xmobot/meshes/camera.dae" scale="1 1 1"/>
+                    </geometry>
+                </xacro:if>
+                <xacro:unless value="${use_mesh}">
+                    <geometry>
+                        <box size="0.05 0.05 0.05"/>
+                    </geometry>
+                </xacro:unless>
                 <material name="Green">
                     <color rgba="0 1 0 1"/>
@@ -37,4 +53,21 @@
             <origin xyz="${camera_offset_x} 0 ${camera_height}" rpy="0 0 0"/>
         </joint>
+        <!-- IMU -->
+        <link name="imu_link">
+            <visual>
+                <origin xyz="0 0 0" rpy="0 0 0"/>
+                <geometry>
+                    <box size="0.05 0.05 0.02"/>
+                </geometry>
+                <material name="Yellow">
+                    <color rgba="1.0 1.0 0.0 1.0"/>
+                </material>
+            </visual>
+        </link>
+        <joint name="imu_joint" type="fixed">
+            <parent link="base_link"/>
+            <child link="imu_link"/>
+            <origin xyz="0 0 0" rpy="0 0 0"/>
+        </joint>
     </xacro:macro>
 </robot>

Commit message: added dual-arm

File: urdf/xmobot.urdf.xacro (robot description, xacro)
@@ -6,11 +6,13 @@
     <xacro:arg name="robot_height" default="0.1"/>
     <xacro:arg name="wheel_radius" default="0.08"/>
-    <xacro:arg name="wheel_width" default="0.02"/>
+    <xacro:arg name="wheel_width" default="0.05"/>
     <xacro:arg name="wheel_separation_x" default="0.5"/>
     <xacro:arg name="wheel_separation_y" default="0.4"/>
     <xacro:arg name="drive_type" default="4wis"/>
     <xacro:arg name="use_mesh" default="false"/>
+    <xacro:arg name="use_arms" default="true"/>
     <!-- 全局参数 -->
     <xacro:property name="use_mesh" value="$(arg use_mesh)"/>
+    <xacro:property name="use_arms" value="$(arg use_arms)"/>
     <xacro:property name="drive_type" value="$(arg drive_type)"/>
     <xacro:property name="robot_length" value="$(arg robot_length)" />
@@ -25,4 +27,17 @@
     <xacro:property name="DEG_TO_RAD" value="0.017453293" />
     <!-- Import Xacro -->
+    <xacro:include filename="$(find xmobot)/urdf/xmobot_inertial.xacro"/>
     <xacro:include filename="$(find xmobot)/urdf/xmobot_base.xacro"/>
+    <xacro:if value="${use_arms}">
+        <xacro:include filename="$(find xmobot)/urdf/xmobot_arm.xacro"/>
+        <xacro:xmobot_arm prefix="left_"  parent_link="base_link" arm_offset_x="0.1"  arm_offset_y="0.145" arm_offset_z="0.0"/>
+        <xacro:xmobot_arm prefix="right_" parent_link="base_link" arm_offset_x="0.1"  arm_offset_y="-0.145" arm_offset_z="0.0"/>
+    </xacro:if>
+    <xacro:include filename="$(find xmobot)/urdf/xmobot_base_gazebo.xacro"/>
+    <xacro:gazebo_base_plugins drive_type="${drive_type}"/>
+    <xacro:include filename="$(find xmobot)/urdf/xmobot_arm_gazebo.xacro"/>
+    <xacro:if value="${use_arms}">
+        <xacro:gazebo_arm_plugins prefix="left_"/>
+        <xacro:gazebo_arm_plugins prefix="right_"/>
+    </xacro:if>
 </robot>

File: urdf/xmobot_base.xacro (robot description, xacro)
@@ -4,6 +4,4 @@
     <xacro:include filename="$(find xmobot)/urdf/xmobot_drive.xacro"/>
     <xacro:include filename="$(find xmobot)/urdf/xmobot_sensors.xacro"/>
-    <xacro:include filename="$(find xmobot)/urdf/xmobot_inertial.xacro"/>
-    <xacro:include filename="$(find xmobot)/urdf/xmobot_gazebo.xacro"/>
     <!-- Basement -->
     <link name="base_footprint"/>
@@ -41,5 +39,3 @@
     <!-- 传感器挂载 -->
     <xacro:sensors/>
-    <!-- gazebo控制接口 -->
-    <xacro:gazebo_plugins/>
 </robot>

File: urdf/xmobot_base_gazebo.xacro (robot description, xacro)
@@ -1,5 +1,5 @@
 <?xml version="1.0"?>
 <robot xmlns:xacro="http://ros.org/wiki/xacro">
-    <xacro:macro name="gazebo_plugins">
+    <xacro:macro name="gazebo_base_plugins" params="drive_type">
         <!-- Gazebo控制器插件 -->
         <gazebo>
@@ -12,5 +12,5 @@
         <!-- Base材质覆盖 -->
         <gazebo reference="base_link">
-            <material>Gazebo/Grey</material>
+            <material>Gazebo/Gray</material>
             <kp>100000.0</kp>
             <kd>1.0</kd>
@@ -140,28 +140,4 @@
             </sensor>
         </gazebo>
-        <!-- 测试用 -->
-        <gazebo reference="front_left_wheel_joint">
-            <implicitSpringDamper>1</implicitSpringDamper>
-        </gazebo>
-        <gazebo reference="front_right_wheel_joint">
-            <implicitSpringDamper>1</implicitSpringDamper>
-        </gazebo>
-        <gazebo reference="rear_left_wheel_joint">
-            <implicitSpringDamper>1</implicitSpringDamper>
-        </gazebo>
-        <gazebo reference="rear_right_wheel_joint">
-            <implicitSpringDamper>1</implicitSpringDamper>
-        </gazebo>
-        <gazebo>
-            <plugin name="object_controller" filename="libgazebo_ros_planar_move.so">
-                <commandTopic>cmd_vel</commandTopic>
-                <odometryTopic>odom</odometryTopic>
-                <odometryFrame>odom</odometryFrame>
-                <odometryRate>20.0</odometryRate>
-                <cmdTimeout>0.25</cmdTimeout>
-                <robotBaseFrame>base_footprint</robotBaseFrame>
-            </plugin>
-        </gazebo>
-        <!-- 测试用 -->
     </xacro:macro>
     <!-- 单个wheel transmission -->
