Commit message: urdf for ros2

File: urdf/xmobot_base_gazebo.xacro (robot description, xacro)
@@ -1,8 +1,8 @@
 <?xml version="1.0"?>
 <robot xmlns:xacro="http://ros.org/wiki/xacro">
-    <xacro:macro name="gazebo_plugins">
+    <xacro:macro name="gazebo_base_plugins" params="drive_type">
         <!-- Gazebo控制器插件 -->
         <gazebo>
-            <plugin name="gazebo_ros_control" filename="libgazebo_ros_control.so">
+            <plugin name="gazebo_ros2_control" filename="libgazebo_ros2_control.so">
                 <robotNamespace>/</robotNamespace>
                 <robotParam>robot_description</robotParam>
@@ -12,5 +12,5 @@
         <!-- Base材质覆盖 -->
         <gazebo reference="base_link">
-            <material>Gazebo/Grey</material>
+            <material>Gazebo/Gray</material>
             <kp>100000.0</kp>
             <kd>1.0</kd>
@@ -62,13 +62,14 @@
         <!-- Lidar仿真 -->
         <gazebo reference="lidar_link">
-            <sensor type="ray" name="lidar_sensor">
+            <sensor name="hls_lfcd_lds" type="ray">
+                <always_on>true</always_on>
+                <visualize>true</visualize>
                 <pose>0 0 0 0 0 0</pose>
-                <visualize>false</visualize>
-                <update_rate>10</update_rate>
+                <update_rate>5</update_rate>
                 <ray>
                     <scan>
                         <horizontal>
                             <samples>360</samples>
-                            <resolution>1</resolution>
+                            <resolution>1.000000</resolution>
                             <min_angle>${-M_PI}</min_angle>
                             <max_angle>${M_PI}</max_angle>
@@ -76,7 +77,7 @@
                     </scan>
                     <range>
-                        <min>0.12</min>
-                        <max>8.0</max>
-                        <resolution>0.001</resolution>
+                        <min>0.120000</min>
+                        <max>8</max>
+                        <resolution>0.015000</resolution>
                     </range>
                     <noise>
@@ -86,7 +87,11 @@
                     </noise>
                 </ray>
-                <plugin name="gazebo_ros_laser_controller" filename="libgazebo_ros_laser.so">
-                    <topicName>scan</topicName>
-                    <frameName>lidar_link</frameName>
+                <plugin name="turtlebot3_laserscan" filename="libgazebo_ros_ray_sensor.so">
+                    <ros>
+                        <!-- <namespace>/tb3</namespace> -->
+                        <remapping>~/out:=scan</remapping>
+                    </ros>
+                    <output_type>sensor_msgs/LaserScan</output_type>
+                    <frame_name>lidar_link</frame_name>
                 </plugin>
             </sensor>
@@ -95,5 +100,7 @@
         <gazebo reference="camera_link">
             <sensor type="camera" name="camera_sensor">
-                <update_rate>10</update_rate>
+                <always_on>true</always_on>
+                <visualize>true</visualize>
+                <update_rate>30</update_rate>
                 <camera>
                     <horizontal_fov>1.39626</horizontal_fov>
@@ -114,8 +121,12 @@
                 </camera>
                 <plugin name="gazebo_ros_camera_controller" filename="libgazebo_ros_camera.so">
-                    <cameraName>camera</cameraName>
-                    <imageTopicName>image_raw</imageTopicName>
-                    <cameraInfoTopicName>camera_info</cameraInfoTopicName>
-                    <frameName>camera_link</frameName>
+                    <ros>
+                        <!-- <namespace>test_cam</namespace> -->
+                        <remapping>image_raw:=image_raw</remapping>
+                        <remapping>camera_info:=camera_info</remapping>
+                    </ros>
+                    <camera_name>camera</camera_name>
+                    <frame_name>camera_link</frame_name>
+                    <hack_baseline>0.07</hack_baseline>
                 </plugin>
             </sensor>
@@ -124,44 +135,58 @@
         <gazebo reference="imu_link">
             <gravity>true</gravity>
-            <sensor type="imu" name="imu_sensor">
+            <sensor name="imu_sensor" type="imu">
                 <always_on>true</always_on>
-                <update_rate>100.0</update_rate>  <!-- 频率可以设置高一点 -->
-                <pose>0 0 0 0 0 0</pose>
+                <update_rate>200</update_rate>
+                <imu>
+                    <angular_velocity>
+                        <x>
+                            <noise type="gaussian">
+                                <mean>0.0</mean>
+                                <stddev>2e-4</stddev>
+                            </noise>
+                        </x>
+                        <y>
+                            <noise type="gaussian">
+                                <mean>0.0</mean>
+                                <stddev>2e-4</stddev>
+                            </noise>
+                        </y>
+                        <z>
+                            <noise type="gaussian">
+                                <mean>0.0</mean>
+                                <stddev>2e-4</stddev>
+                            </noise>
+                        </z>
+                    </angular_velocity>
+                    <linear_acceleration>
+                        <x>
+                            <noise type="gaussian">
+                                <mean>0.0</mean>
+                                <stddev>1.7e-2</stddev>
+                            </noise>
+                        </x>
+                        <y>
+                            <noise type="gaussian">
+                                <mean>0.0</mean>
+                                <stddev>1.7e-2</stddev>
+                            </noise>
+                        </y>
+                        <z>
+                            <noise type="gaussian">
+                                <mean>0.0</mean>
+                                <stddev>1.7e-2</stddev>
+                            </noise>
+                        </z>
+                    </linear_acceleration>
+                </imu>
                 <plugin name="gazebo_ros_imu" filename="libgazebo_ros_imu_sensor.so">
-                    <bodyName>imu_link</bodyName>
-                    <topicName>imu/data</topicName>
-                    <updateRateHZ>100.0</updateRateHZ>
-                    <gaussianNoise>0.0</gaussianNoise>
-                    <xyzOffset>0 0 0</xyzOffset>
-                    <rpyOffset>0 0 0</rpyOffset>
-                    <frameName>imu_link</frameName>
-                    <initialOrientationAsReference>false</initialOrientationAsReference>
+                    <ros>
+                        <!-- <namespace>/xmobot</namespace> -->
+                        <remapping>~/out:=imu</remapping>
+                    </ros>
+                    <initial_orientation_as_reference>false</initial_orientation_as_reference>>
                 </plugin>
             </sensor>
         </gazebo>
-        <!-- 测试用 -->
-        <gazebo reference="front_left_wheel_joint">
-            <implicitSpringDamper>1</implicitSpringDamper>
-        </gazebo>
-        <gazebo reference="front_right_wheel_joint">
-            <implicitSpringDamper>1</implicitSpringDamper>
-        </gazebo>
-        <gazebo reference="rear_left_wheel_joint">
-            <implicitSpringDamper>1</implicitSpringDamper>
-        </gazebo>
-        <gazebo reference="rear_right_wheel_joint">
-            <implicitSpringDamper>1</implicitSpringDamper>
-        </gazebo>
-        <gazebo>
-            <plugin name="object_controller" filename="libgazebo_ros_planar_move.so">
-                <commandTopic>cmd_vel</commandTopic>
-                <odometryTopic>odom</odometryTopic>
-                <odometryFrame>odom</odometryFrame>
-                <odometryRate>20.0</odometryRate>
-                <cmdTimeout>0.25</cmdTimeout>
-                <robotBaseFrame>base_footprint</robotBaseFrame>
-            </plugin>
-        </gazebo>
-        <!-- 测试用 -->
     </xacro:macro>
     <!-- 单个wheel transmission -->
